Commit message: initial setup for buggy

File: config/robot.urdf.xacro (robot description, xacro)
@@ -9,9 +9,21 @@
     <origin xyz="0 0 0" rpy="0 0 0" />
   </joint>
-  <link name="lidar_link"> </link>
-  <joint name="lidar_joint" type="fixed">
+  <link name="velodyne_top"> </link>
+  <joint name="lidar_joint_top" type="fixed">
     <parent link="base_link" />
-    <child link="lidar_link" />
-    <origin xyz="0 0 0" rpy="0 0 0" />
+    <child link="velodyne_top" />
+    <origin xyz="-0.478 0.0125 1.952" rpy="0 0 3.14159265359" />
+  </joint>
+  <link name="velodyne_left"> </link>
+  <joint name="lidar_joint_left" type="fixed">
+    <parent link="base_link" />
+    <child link="velodyne_left" />
+    <origin xyz="3.25 0.55 0.825" rpy="0 0 0" />
+  </joint>
+  <link name="velodyne_right"> </link>
+  <joint name="lidar_joint_right" type="fixed">
+    <parent link="base_link" />
+    <child link="velodyne_right" />
+    <origin xyz="3.25 -0.55 0.825" rpy="0 0 0" />
   </joint>
   <link name="imu_link"> </link>
@@ -19,5 +31,5 @@
     <parent link="chassis_link" />
     <child link="imu_link" />
-    <origin xyz="0 0 0" rpy="0 0 0" />
+    <origin xyz="-0.2 0 0" rpy="0 0 0" />
   </joint>
   <link name="laser_sensor_frame"> </link>
@@ -31,5 +43,5 @@
     <parent link="chassis_link" />
     <child link="navsat_link" />
-    <origin xyz="0 0 0" rpy="0 0 0" />
+    <origin xyz="0.5 0 1.952" rpy="0 0 0" />
   </joint>
 </robot>

Commit message: update imu tf

File: config/robot.urdf.xacro (robot description, xacro)
@@ -31,5 +31,5 @@
     <parent link="chassis_link" />
     <child link="imu_link" />
-    <origin xyz="-0.2 0 0" rpy="0 0 0" />
+    <origin xyz="-0.2 0 0.8" rpy="0 0 0" />
   </joint>
   <link name="laser_sensor_frame"> </link>
